File: arduino_uno.sch (KiCad schematic (older format))
At the start: 42 parts, among them J1 Barrel_Jack_Switch, J2 USB_B, J3 Conn_01x04, J4 Conn_01x06, J5 Conn_01x08, J6 Conn_01x06, J7 Conn_01x08, Q1 KIA3401, SW1 SW_Push, U1 LM393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

Commit message: Se agrega to-do, mejoras esteticas para legibilidad
Parts:
- removed R3: R_US, symbol Device:R_US
- added R6: 1k, symbol Device:R_US
- D1: value D -> Schottky
- D2: value LED -> Azul
- D3: value LED -> Verde
- D4, D5: value LED -> Rojo
- J1: value Barrel_Jack_Switch -> DC_IN
- J2: value USB_B -> USB
- J3: value Conn_01x04 -> A6,7
- J4: value Conn_01x06 -> Power
- J5: value Conn_01x08 -> D8-13
- J6: value Conn_01x06 -> A0-5
- J7: value Conn_01x08 -> D0-7
- U3: value CH340G -> CH340G/C
- renumbered R4 to R3, R5 to R4, R6 to R5
Connections:
- net at U1.6 (_), U1.7: now also R6.2
- net at D2.2 (A): now also R6.1
Other:
- note added: "Por hacer:\nFusible en VCCUSB\nPuerto ICSP\nHeader I2C\nFerritas en D+/D-\nTransistores en LEDs TX/RX"
- moved on the sheet: C1, C4, C5, C6, C8, D3, D4, D5, Q1, R1, R2, R3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

Commit message: Se agregan ICSP e I2C, varias mejoras para legibilidad
Parts:
- removed D1: Schottky, symbol Device:D
- added D2: D_Schottky, symbol Device:D_Schottky
- added F1: Polyfuse, Fuse:Fuse_1206_3216Metric, symbol Device:Polyfuse
- added J2: ICSP, Connector_PinHeader_2.54mm:PinHeader_2x03_P2.54mm_Vertical, symbol Connector_Generic:Conn_02x03_Odd_Even
- added J6: I2C, Connector_PinSocket_2.54mm:PinSocket_1x04_P2.54mm_Vertical, symbol Connector_Generic:Conn_01x04
- C1: renamed from C4; footprint (none) -> Capacitor_SMD:CP_Elec_6.3x5.4
- C10: renamed from C9; footprint (none) -> Capacitor_SMD:C_0603_1608Metric
- C11: renamed from C2; footprint (none) -> Capacitor_SMD:C_0603_1608Metric
- C12: renamed from C3; footprint (none) -> Capacitor_SMD:C_0603_1608Metric
- C13: renamed from C11; footprint (none) -> Capacitor_SMD:C_0603_1608Metric
- C14: renamed from C13; footprint (none) -> Capacitor_SMD:C_0603_1608Metric
- C2: renamed from C6; footprint (none) -> Capacitor_SMD:CP_Elec_6.3x5.4
- C3: renamed from C7; footprint (none) -> Capacitor_SMD:C_0603_1608Metric
- C4: renamed from C10; footprint (none) -> Capacitor_SMD:C_0603_1608Metric
- C5: renamed from C14; footprint (none) -> Capacitor_SMD:C_0603_1608Metric
- C6: renamed from C1; footprint (none) -> Capacitor_SMD:C_0603_1608Metric
- C7: renamed from C12; footprint (none) -> Capacitor_SMD:C_0603_1608Metric
- C8: renamed from C5; footprint (none) -> Capacitor_SMD:C_0603_1608Metric
- C9: renamed from C8; footprint (none) -> Capacitor_SMD:C_0603_1608Metric
- D1: renamed from D3; footprint (none) -> LED_SMD:LED_0603_1608Metric
- D3: renamed from D4; footprint (none) -> LED_SMD:LED_0603_1608Metric
- D4: renamed from D5; footprint (none) -> LED_SMD:LED_0603_1608Metric
- D5: renamed from D2; footprint (none) -> LED_SMD:LED_0603_1608Metric
- J1: footprint (none) -> Connector_BarrelJack:BarrelJack_Horizontal
- J3: renamed from J4; footprint (none) -> Connector_PinSocket_2.54mm:PinSocket_1x06_P2.54mm_Vertical
- J4: renamed from J3; footprint (none) -> Connector_PinSocket_2.54mm:PinSocket_1x04_P2.54mm_Vertical
- J5: footprint (none) -> Connector_PinSocket_2.54mm:PinSocket_1x08_P2.54mm_Vertical
- J7: renamed from J6; footprint (none) -> Connector_PinSocket_2.54mm:PinSocket_1x06_P2.54mm_Vertical
- J9: renamed from J7; footprint (none) -> Connector_PinSocket_2.54mm:PinSocket_1x08_P2.54mm_Vertical
- Q1: footprint (none) -> Package_TO_SOT_SMD:SOT-23
- R1: renamed from R3; footprint (none) -> Resistor_SMD:R_0603_1608Metric
- R2: renamed from R4; footprint (none) -> Resistor_SMD:R_0603_1608Metric
- R3: renamed from R5; footprint (none) -> Resistor_SMD:R_0603_1608Metric
- R4: renamed from R6; footprint (none) -> Resistor_SMD:R_0603_1608Metric
- R5: renamed from R1; footprint (none) -> Resistor_SMD:R_0603_1608Metric
- R6: renamed from R2; footprint (none) -> Resistor_SMD:R_0603_1608Metric
- R7: footprint (none) -> Resistor_SMD:R_0603_1608Metric
- U1: renamed from U2; footprint (none) -> Package_TO_SOT_SMD:SOT-223-3_TabPin2
- U3: renamed from U1; footprint (none) -> Package_SO:SOIC-8_3.9x4.9mm_P1.27mm
- Y2: footprint (none) -> Crystal:Crystal_SMD_SeikoEpson_TSX3225-4Pin_3.2x2.5mm
- renumbered J2 to J8, U4 to U2, U5 to U4, U3 to U5
Connections:
- net 5V: now also J6.2 (Pin_2)
- net A4: now also J6.3 (Pin_3)
- net A5: now also J6.4 (Pin_4)
- net D11: now also J2.4 (Pin_4)
- net D12: now also J2.1 (Pin_1)
- net D13: now also J2.3 (Pin_3)
- net GND: now also J2.6 (Pin_6), J6.1 (Pin_1)
- net RAW: now also D2.1 (K)
- net RST: now also J2.5 (Pin_5)
- net at J1.1: now also D2.2 (A)
- net at J8.1 (VBUS): now also F1.2; no longer Q1.2 (S)
- new net: F1.1, Q1.2 (S)
- new net VCC: J2.2 (Pin_2)
Other:
- note added: "MISO\nSCK"
- note added: "MOSI"
- note added: "Por hacer:\nFerritas en D+/D-\nTransistores en LEDs TX/RX"
- note added: "SCL\nSDA"
- note removed: "Por hacer:\nFusible en VCCUSB\nPuerto ICSP\nHeader I2C\nFerritas en D+/D-\nTransistores en LEDs TX/RX"
- moved on the sheet: C13, C14, C6, Q1, R5, R6, SW1, U3A, U3B, U3C, Y2

Commit message: Primera revision completa, se fabrica para evaluacion
Parts:
- removed Y1: Crystal, symbol Device:Crystal
- added Y1: Crystal_GND3, protoplasma:Crystal_DS26_D2.0mm_L6.0mm_Horizontal_Grounded, symbol Device:Crystal_GND3
- D2: footprint (none) -> Diode_SMD:D_SMA
- J8: footprint (none) -> Connector_USB:USB_B_OST_USB-B1HSxx_Horizontal
- SW1: footprint (none) -> protoplasma:Switch_SMD_4545
- U5: footprint Package_SO:SOIC-16_3.9x9.9mm_P1.27mm -> Package_SO:SOP-16_4.4x10.4mm_P1.27mm
Connections:
- net VCC is gone; now on net 5V: J2.2 (Pin_2)
- net GND: now also Y1.3
- net at C11.1, U5.7 (XI): now also Y1.1
- net at C12.1, U5.8 (XO): now also Y1.2
Other:
- moved on the sheet: C12
Changed lines of the file:
@@
 EESchema Schematic File Version 4
 LIBS:arduino_uno-cache
-EELAYER 29 0
+EELAYER 26 0
 EELAYER END
 $Descr A4 11693 8268
@@
 F 0 "J8" H 2305 5367 50  0000 C CNN
 F 1 "USB" H 2305 5276 50  0000 C CNN
-F 2 "" H 2400 4850 50  0001 C CNN
+F 2 "Connector_USB:USB_B_OST_USB-B1HSxx_Horizontal" H 2400 4850 50  0001 C CNN
 F 3 " ~" H 2400 4850 50  0001 C CNN
 	1    2250 4900
@@
 F 0 "U5" H 4400 4314 50  0000 C CNN
 F 1 "CH340G/C" H 4400 4223 50  0000 C CNN
-F 2 "Package_SO:SOIC-16_3.9x9.9mm_P1.27mm" H 4450 4450 50  0001 L CNN
+F 2 "Package_SO:SOP-16_4.4x10.4mm_P1.27mm" H 4450 4450 50  0001 L CNN
 F 3 "http://www.datasheet5.com/pdf-local-2195953" H 4050 5800 50  0001 C CNN
 	1    4400 5000
@@
 	4400 5600 4400 5850
 Wire Wire Line
-	4400 5850 3450 5850
+	4400 5850 3550 5850
 Connection ~ 2250 5850
 Wire Wire Line
@@
 Wire Wire Line
 	4150 3200 4350 3200
-$Comp
-L Device:Crystal Y1
-U 1 1 5D2E6FFC
-P 3200 5400
-F 0 "Y1" H 3200 5668 50  0000 C CNN
-F 1 "Crystal" H 3200 5577 50  0000 C CNN
-F 2 "" H 3200 5400 50  0001 C CNN
-F 3 "~" H 3200 5400 50  0001 C CNN
-	1    3200 5400
-	1    0    0    -1
-$EndComp
-Wire Wire Line
-	4000 5400 3450 5400
+Wire Wire Line
+	4000 5400 3550 5400
 Wire Wire Line
 	4000 5200 2950 5200
@@
 	2950 5200 2950 5400
 Wire Wire Line
-	2950 5400 3050 5400
+	2950 5400 3100 5400
 $Comp
 L Regulator_Linear:APE8865N-33-HF-3 U2
@@
 L Device:C_Small C12
 U 1 1 5D47E07A
-P 3450 5650
-F 0 "C12" H 3542 5696 50  0000 L CNN
-F 1 "15p" H 3542 5605 50  0000 L CNN
-F 2 "Capacitor_SMD:C_0603_1608Metric" H 3450 5650 50  0001 C CNN
-F 3 "~" H 3450 5650 50  0001 C CNN
-	1    3450 5650
-	1    0    0    -1
-$EndComp
-Wire Wire Line
-	3450 5550 3450 5400
-Connection ~ 3450 5400
-Wire Wire Line
-	3450 5400 3350 5400
+P 3550 5650
+F 0 "C12" H 3642 5696 50  0000 L CNN
+F 1 "15p" H 3642 5605 50  0000 L CNN
+F 2 "Capacitor_SMD:C_0603_1608Metric" H 3550 5650 50  0001 C CNN
+F 3 "~" H 3550 5650 50  0001 C CNN
+	1    3550 5650
+	1    0    0    -1
+$EndComp
+Wire Wire Line
+	3550 5550 3550 5400
+Connection ~ 3550 5400
+Wire Wire Line
+	3550 5400 3400 5400
 Wire Wire Line
 	2950 5550 2950 5400
@@
 	2950 5850 2250 5850
 Wire Wire Line
-	3450 5750 3450 5850
-Connection ~ 3450 5850
-Wire Wire Line
-	3450 5850 2950 5850
+	3550 5750 3550 5850
+Connection ~ 3550 5850
+Wire Wire Line
+	3550 5850 3250 5850
 Connection ~ 4800 2100
 Wire Wire Line
@@
 F 0 "D2" H 2700 2016 50  0000 C CNN
 F 1 "D_Schottky" H 2700 1925 50  0000 C CNN
-F 2 "" H 2700 1800 50  0001 C CNN
+F 2 "Diode_SMD:D_SMA" H 2700 1800 50  0001 C CNN
 F 3 "~" H 2700 1800 50  0001 C CNN
 	1    2700 1800
@@
 F 0 "SW1" H 7050 5185 50  0000 C CNN
 F 1 "SW_Push" H 7050 5094 50  0000 C CNN
-F 2 "" H 7050 5100 50  0001 C CNN
+F 2 "protoplasma:Switch_SMD_4545" H 7050 5100 50  0001 C CNN
 F 3 "" H 7050 5100 50  0001 C CNN
 	1    7050 4900
@@
 D12
 Text GLabel 8800 1800 2    50   Input ~ 0
-VCC
+5V
 $Comp
 L power:GND #PWR02
@@
 Wire Wire Line
 	3050 4700 3300 4700
+$Comp
+L Device:Crystal_GND3 Y1
+U 1 1 5D32C52B
+P 3250 5400
+F 0 "Y1" H 3250 5668 50  0000 C CNN
+F 1 "Crystal_GND3" H 3250 5577 50  0000 C CNN
+F 2 "protoplasma:Crystal_DS26_D2.0mm_L6.0mm_Horizontal_Grounded" H 3250 5400 50  0001 C CNN
+F 3 "~" H 3250 5400 50  0001 C CNN
+	1    3250 5400
+	1    0    0    -1
+$EndComp
+Wire Wire Line
+	3250 5600 3250 5850
+Connection ~ 3250 5850
+Wire Wire Line
+	3250 5850 2950 5850
 $EndSCHEMATC
